File: sd-card.kicad_sch (KiCad schematic)
At the start: 3 parts, among them J12 Micro_SD_Card

Commit message: update schematics and add 3d models
Parts:
- C3: footprint (none) -> Capacitor_SMD:C_0402_1005Metric; LCSC (none) -> C15525
- J12: LCSC (none) -> C164170
Changed lines of the file:
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@@
+			)
+		)
+		(property "LCSC" "C164170"
+			(at 139.7 82.55 0)
+			(effects
+				(font
+					(size 1.27 1.27)
+				)
+				(hide yes)
 			)
 		)
@@
 			)
 		)
-		(property "Footprint" ""
+		(property "Footprint" "Capacitor_SMD:C_0402_1005Metric"
 			(at 113.03 63.5 0)
 			(effects
@@
 			)
 		)
+		(property "LCSC" "C15525"
+			(at 113.03 63.5 0)
+			(effects
+				(font
+					(size 1.27 1.27)
+				)
+				(hide yes)
+			)
+		)
 		(pin "1"
 		)
@@
 			(at 95.25 97.79 0)
 			(effects
+				(font
+					(size 1.27 1.27)
+				)
+				(hide yes)
+			)
+		)
+		(property "LCSC" ""
+			(at 95.25 97.79 0)
+			(effects
