File: sd-card.kicad_sch (KiCad schematic)
At the start: 3 parts, among them J12 Micro_SD_Card

Commit message: final tweaks, as sent to fab
Changed lines of the file:
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@@
 	(wire
 		(pts
-			(xy 113.03 57.15) (xy 113.03 59.69)
+			(xy 113.03 58.42) (xy 113.03 59.69)
 		)
 		(stroke
@@
 	(symbol
 		(lib_id "power:+3V3")
-		(at 113.03 57.15 0)
+		(at 113.03 58.42 0)
 		(unit 1)
 		(body_style 1)
@@
 		(fields_autoplaced yes)
 		(property "Reference" "#PWR052"
-			(at 113.03 60.96 0)
+			(at 113.03 62.23 0)
 			(hide yes)
 			(show_name no)
@@
 		)
 		(property "Value" "+3V3"
-			(at 113.03 52.07 0)
+			(at 113.03 53.34 0)
 			(show_name no)
 			(do_not_autoplace no)
@@
 		)
 		(property "Footprint" ""
-			(at 113.03 57.15 0)
+			(at 113.03 58.42 0)
 			(hide yes)
 			(show_name no)
@@
 		)
 		(property "Datasheet" ""
-			(at 113.03 57.15 0)
+			(at 113.03 58.42 0)
 			(hide yes)
 			(show_name no)
@@
 		)
 		(property "Description" "Power symbol creates a global label with name \"+3V3\""
-			(at 113.03 57.15 0)
-			(hide yes)
-			(show_name no)
+			(at 113.03 58.42 0)
+			(hide yes)
+			(show_name no)
