File: beavs-6.kicad_sch (KiCad schematic)
At the start: 16 parts, among them J1 USB_C_Receptacle_USB2.0_16P, J5 Conn_01x02, U15 SN74LVC4245APW, U16 SRV05-4, U17 SRV05-4

Commit message: add schematic PDF, improve schematic readability
Other:
- sheet mcu ports: added GPS_EXTINT; removed GPIO_EXTINT
- note added: "Active high; must be held low on startup to limit inrush current"
- note added: "Baro"
- note added: "IMU"
- note added: "Magn"
- note added: "Radio"
- note added: "SD"
- note added: "Status"
Changed lines of the file:
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@@
 	(generator_version "9.0")
 	(paper "A3")
+	(text "Baro"
+		(exclude_from_sim no)
+		(at 352.552 156.718 0)
+		(effects
+			(font
+				(size 1.27 1.27)
+			)
+		)
+	)
+	(text "SD"
+		(exclude_from_sim no)
+		(at 302.768 156.972 0)
+		(effects
+			(font
+				(size 1.27 1.27)
+			)
+		)
+	)
+	(text "IMU"
+		(exclude_from_sim no)
+		(at 336.55 156.718 0)
+		(effects
+			(font
+				(size 1.27 1.27)
+			)
+		)
+	)
+	(text "Radio"
+		(exclude_from_sim no)
+		(at 319.532 156.718 0)
+		(effects
+			(font
+				(size 1.27 1.27)
+			)
+		)
+	)
+	(text "Status"
+		(exclude_from_sim no)
+		(at 384.81 156.972 0)
+		(effects
+			(font
+				(size 1.27 1.27)
+			)
+		)
+	)
+	(text "Active high; must be held low on\nstartup to limit inrush current"
+		(exclude_from_sim no)
+		(at 132.842 131.826 0)
+		(effects
+			(font
+				(size 1.27 1.27)
+			)
+		)
+	)
+	(text "Magn"
+		(exclude_from_sim no)
+		(at 368.554 156.718 0)
+		(effects
+			(font
+				(size 1.27 1.27)
+			)
+		)
+	)
 	(junction
 		(at 271.78 142.24)
@@
 		)
 		(instances
-			(project "beavs-sketch-0"
+			(project "beavs-6"
 				(path "/49232f62-a438-4b3e-9be5-c2b3074d8de1"
 					(page "6")
@@
 			)
 		)
-		(pin "GPIO_EXTINT" output
+		(pin "GPS_EXTINT" output
 			(at 223.52 69.85 0)
 			(effects
@@
 		)
 		(instances
-			(project "beavs-sketch-0"
+			(project "beavs-6"
 				(path "/49232f62-a438-4b3e-9be5-c2b3074d8de1"
 					(page "2")
@@
 		)
 		(instances
-			(project "beavs-sketch-0"
+			(project "beavs-6"
 				(path "/49232f62-a438-4b3e-9be5-c2b3074d8de1"
 					(page "7")
@@
 		)
 		(instances
-			(project "beavs-sketch-0"
+			(project "beavs-6"
 				(path "/49232f62-a438-4b3e-9be5-c2b3074d8de1"
 					(page "5")
@@
 		)
 		(instances
-			(project "beavs-sketch-0"
+			(project "beavs-6"
 				(path "/49232f62-a438-4b3e-9be5-c2b3074d8de1"
 					(page "3")
@@
 		)
 		(instances
-			(project "beavs-sketch-0"
+			(project "beavs-6"
 				(path "/49232f62-a438-4b3e-9be5-c2b3074d8de1"
 					(page "4")
