File: beavs-6.kicad_sch (KiCad schematic)
At the start: 16 parts, among them J1 USB_C_Receptacle_USB2.0_16P, J5 Conn_01x02, U15 SN74LVC4245APW, U16 SRV05-4, U17 SRV05-4

Commit message: remove unneeded stuff
Connections:
- net mcu/M_S6 is gone; now on net GND: U15.20 (B2)
- net servos/S6: no longer names the net of U17.1 (IO1)
- net servos/S6: no longer U15.4 (A2)
- no-connect marks 4 -> 5
Other:
- removed sheet Radio
- sheet Sensors ports: added none; removed EXTINT
- sheet mcu ports: added none; removed GPS_EXTINT, M_S6, RADIO_CS, RADIO_D0, RADIO_RESET
- sheet servos ports: added none; removed S6

Commit message: changes!
Parts:
- added JP1: Jumper_2_Open, Resistor_SMD:R_0402_1005Metric, symbol Jumper:Jumper_2_Open
Connections:
- net +5V: now also JP1.2 (B)
- net VBUS: now also JP1.1 (A)
- net mcu/M_S1: now also U15.19 (B3); no longer U15.15 (B7)
- net mcu/M_S2: now also U15.18 (B4); no longer U15.16 (B6)
- net mcu/M_S4: now also U15.16 (B6); no longer U15.18 (B4)
- net mcu/M_S5: now also U15.15 (B7); no longer U15.19 (B3)
- net servos/S1: now also U15.5 (A3), U17.6 (IO4); no longer U15.9 (A7), U16.1 (IO1)
- net servos/S2: now also U15.6 (A4), U17.3 (IO2); no longer U15.8 (A6), U16.3 (IO2)
- net servos/S4: now also U15.8 (A6), U16.3 (IO2); no longer U15.6 (A4), U17.3 (IO2)
- net servos/S5: now also U15.9 (A7), U16.1 (IO1); no longer U15.5 (A3), U17.6 (IO4)
Other:
- note removed: "Active high; must be held low on startup to limit inrush current"

Commit message: relayout and route
Parts:
- removed D6: SK6812-EC20, beavs-footprints:LED_SK6812-EC20_PLCC4_2.0x2.0mm, symbol beavs-symbols:SK6812-EC20
- removed U16, U17: SRV05-4, Package_TO_SOT_SMD:SOT-23-6, symbol Power_Protection:SRV05-4
Connections:
- net mcu/M_S1: now also U15.15 (B7); no longer U15.19 (B3)
- net mcu/M_S2: now also U15.16 (B6); no longer U15.18 (B4)
- net mcu/M_S4: now also U15.18 (B4); no longer U15.16 (B6)
- net mcu/M_S5: now also U15.19 (B3); no longer U15.15 (B7)
- net servos/S1: now also U15.9 (A7); no longer U15.5 (A3)
- net servos/S2: now also U15.8 (A6); no longer U15.6 (A4)
- net servos/S4: now also U15.6 (A4); no longer U15.8 (A6)
- net servos/S5: now also U15.5 (A3); no longer U15.9 (A7)
- net +BATT renamed VDD
Other:
- note removed: "Radio"

Commit message: restore symbols library, wire up PG and IMON, refine routing
Other:
- sheet Power ports: added IMON, PG; removed none
- sheet mcu ports: added IMON, PG; removed none
Changed lines of the file:
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@@
 	(wire
 		(pts
+			(xy 96.52 138.43) (xy 171.45 138.43)
+		)
+		(stroke
+			(width 0)
+			(type default)
+		)
+	)
+	(wire
+		(pts
 			(xy 158.75 189.23) (xy 158.75 187.96)
 		)
@@
 	(wire
 		(pts
+			(xy 96.52 140.97) (xy 171.45 140.97)
+		)
+		(stroke
+			(width 0)
+			(type default)
+		)
+	)
+	(wire
+		(pts
 			(xy 299.72 158.75) (xy 299.72 160.02)
 		)
@@
 			)
 		)
+		(pin "IMON" input
+			(at 171.45 138.43 180)
+			(effects
+				(font
+					(size 1.27 1.27)
+				)
+				(justify left)
+			)
+		)
+		(pin "PG" input
+			(at 171.45 140.97 180)
+			(effects
+				(font
+					(size 1.27 1.27)
+				)
+				(justify left)
+			)
+		)
 		(instances
 			(project "beavs-6"
@@
 			(effects
 				(font
+					(size 1.27 1.27)
+				)
+				(justify right)
+			)
+		)
+		(pin "IMON" output
+			(at 96.52 138.43 0)
+			(effects
+				(font
+					(size 1.27 1.27)
+				)
+				(justify right)
+			)
+		)
+		(pin "PG" output
+			(at 96.52 140.97 0)
+			(effects
+				(font

Commit message: mostly cosmetic changes
Parts:
- added R17, R18: 56k, Resistor_SMD:R_0402_1005Metric, symbol Device:R_Small
Connections:
- net +5V: now also R17.1, R18.1
- net mcu/M_S2: now also U15.19 (B3); no longer U15.16 (B6)
- net mcu/M_S3: now also U15.18 (B4); no longer U15.17 (B5)
- net mcu/M_S4: now also U15.17 (B5); no longer U15.18 (B4)
- net mcu/M_S5: now also U15.16 (B6); no longer U15.19 (B3)
- net servos/S2: now also U15.5 (A3); no longer U15.8 (A6)
- net servos/S3: now also U15.6 (A4); no longer U15.7 (A5)
- net servos/S4: now also U15.7 (A5); no longer U15.6 (A4)
- net servos/S5: now also U15.8 (A6); no longer U15.5 (A3)
- net at J1.A5 (CC1), R3.1: now also R17.2
- net at J1.B5 (CC2), R5.1: now also R18.2
Other:
- note added: "Add jumper, remove 5.1k resistors, add 56k resistors for USB host"
- moved on the sheet: D1, D2, D3, D4, D5, JP1, R3, R5

Commit message: final tweaks, as sent to fab
Parts:
- added D10, D11, D17, D18, D6: D_Zener, Diode_SMD:D_SOD-523, symbol Device:D_Zener
Connections:
- net GND: now also D10.2 (A), D11.2 (A), D17.2 (A), D18.2 (A), D6.2 (A)
- net servos/S1: now also D6.1 (K)
- net servos/S2: now also D18.1 (K)
- net servos/S3: now also D17.1 (K)
- net servos/S4: now also D11.1 (K)
- net servos/S5: now also D10.1 (K)
