File: mcu.kicad_sch (KiCad schematic)
At the start: 28 parts, among them J13 Conn_02x02_Odd_Even, J14 Conn_01x02, SW1 SW_Push, SW2 SW_Push, U1 RP2040, U2 W25Q128JVS, Y1 Crystal_GND24

Commit message: remove unneeded stuff
Parts:
- removed J13: Conn_02x02_Odd_Even, Connector_PinHeader_1.27mm:PinHeader_2x02_P1.27mm_Vertical, symbol Connector_Generic:Conn_02x02_Odd_Even
- removed TP1, TP2: TestPoint, TestPoint:TestPoint_Pad_D1.0mm, symbol Connector:TestPoint
- added J2: Conn_ARM_JTAG_SWD_10, Connector_PinHeader_1.27mm:PinHeader_2x05_P1.27mm_Vertical_SMD, symbol Connector:Conn_ARM_JTAG_SWD_10
- added J4: Conn_01x04, Connector_JST:JST_PH_B4B-PH-K_1x04_P2.00mm_Vertical, symbol Connector_Generic:Conn_01x04
Connections:
- net +3V3: now also J2.1 (VTref), J4.1 (Pin_1)
- net GND: now also J2.3 (GND), J2.5 (GND), J4.4 (Pin_4)
- net MISO: no longer U1.13 (GPIO10)
- net MOSI: no longer U1.12 (GPIO9)
- net SCK: no longer U1.14 (GPIO11)
- net ~{RESET}: now also J2.10 (~{RESET})
- net at U1.24 (SWCLK): now also J2.4 (SWCLK/TCK)
- net at U1.25 (SWD): now also J2.2 (SWDIO/TMS)
- net EXPANSION_1: no longer names the net of U1.9 (GPIO7)
- net EXPANSION_2: no longer names the net of U1.18 (GPIO15)
- net GPS_EXTINT: no longer names the net of U1.39 (GPIO27_ADC1)
- net M_S6: no longer names the net of U1.27 (GPIO16)
- net RADIO_CS: no longer names the net of U1.2 (GPIO0)
- net RADIO_D0: no longer names the net of U1.3 (GPIO1)
- net RADIO_RESET: no longer names the net of U1.4 (GPIO2)
- no-connect marks 0 -> 2
