File: mcu.kicad_sch (KiCad schematic)
At the start: 27 parts, among them J14 Conn_01x02, J2 Conn_ARM_JTAG_SWD_10, J4 Conn_01x04, SW1 SW_Push, SW2 SW_Push, U1 RP2040, U2 W25Q128JVS, Y1 Crystal_GND24

Commit message: changes!
Connections:
- net ARM_SWITCH: no longer U1.8 (GPIO6)
- net BARO_CS: now also U1.3 (GPIO1); no longer U1.16 (GPIO13)
- net BATTERY_SENSE: now also U1.41 (GPIO29_ADC3); no longer U1.38 (GPIO26_ADC0)
- net IMU_CS: now also U1.8 (GPIO6); no longer U1.17 (GPIO14)
- net LEVELSHIFT_DIR: now also U1.34 (GPIO22); no longer U1.5 (GPIO3)
- net MISO: now also U1.2 (GPIO0)
- net MOSI: now also U1.5 (GPIO3)
- net M_LED_D: now also U1.35 (GPIO23); no longer U1.15 (GPIO12)
- net M_S1: now also U1.36 (GPIO24); no longer U1.40 (GPIO28_ADC2)
- net M_S2: now also U1.37 (GPIO25); no longer U1.41 (GPIO29_ADC3)
- net M_S3: now also U1.38 (GPIO26_ADC0); no longer U1.37 (GPIO25)
- net M_S4: now also U1.39 (GPIO27_ADC1); no longer U1.36 (GPIO24)
- net M_S5: now also U1.40 (GPIO28_ADC2); no longer U1.28 (GPIO17)
- net SCK: now also U1.4 (GPIO2)
- net SD_CLK: now also U1.15 (GPIO12); no longer U1.35 (GPIO23)
- net SD_CMD: now also U1.9 (GPIO7); no longer U1.29 (GPIO18)
- net SD_DAT0: now also U1.11 (GPIO8); no longer U1.30 (GPIO19)
- net SD_DAT1: now also U1.12 (GPIO9); no longer U1.31 (GPIO20)
- net SD_DAT2: now also U1.13 (GPIO10); no longer U1.32 (GPIO21)
- net SD_DAT3: now also U1.14 (GPIO11); no longer U1.34 (GPIO22)
- net SERVO_POWER_EN: no longer U1.11 (GPIO8)

Commit message: relayout and route
Parts:
- added C22: 100n, Capacitor_SMD:C_0402_1005Metric, symbol Device:C_Small
Connections:
- net +3V3: now also C22.1
- net ARM_SWITCH: now also U1.40 (GPIO28_ADC2)
- net GND: now also C22.2
- net LEVELSHIFT_DIR: now also U1.29 (GPIO18); no longer U1.34 (GPIO22)
- net M_LED_D: now also U1.34 (GPIO22); no longer U1.35 (GPIO23)
- net M_S1: now also U1.39 (GPIO27_ADC1); no longer U1.36 (GPIO24)
- net M_S2: now also U1.38 (GPIO26_ADC0); no longer U1.37 (GPIO25)
- net M_S3: now also U1.37 (GPIO25); no longer U1.38 (GPIO26_ADC0)
- net M_S4: now also U1.36 (GPIO24); no longer U1.39 (GPIO27_ADC1)
- net M_S5: now also U1.35 (GPIO23); no longer U1.40 (GPIO28_ADC2)
- net SERVO_POWER_EN: now also U1.28 (GPIO17)
- net at J4.2 (Pin_2): now also U1.17 (GPIO14)
- net at J4.3 (Pin_3): now also U1.18 (GPIO15)
Other:
- moved on the sheet: J4

Commit message: add reverse polarity protection
Connections:
- net ARM_SWITCH: now also U1.32 (GPIO21); no longer U1.40 (GPIO28_ADC2)
- new net IMON: U1.40 (GPIO28_ADC2)

Commit message: restore symbols library, wire up PG and IMON, refine routing
Connections:
- net PG: now reaches U1.30 (GPIO19)
Changed lines of the file:
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@@
+	(wire
+		(pts
+			(xy 193.04 92.71) (xy 198.12 92.71)
+		)
+		(stroke
+			(width 0)
+			(type default)
+		)
+	)
 	(wire
 		(pts
@@
 		(effects
 			(font
+				(size 1.27 1.27)
+			)
+			(justify left)
+		)
+	)
+	(hierarchical_label "PG"
+		(shape input)
+		(at 198.12 92.71 0)
+		(effects
+			(font

Commit message: mostly cosmetic changes
Parts:
- added J11: Conn_01x03, Connector_PinHeader_2.54mm:PinHeader_1x03_P2.54mm_Vertical, symbol Connector_Generic:Conn_01x03
Connections:
- net GND: now also J11.3 (Pin_3)
- net M_S2: now also U1.35 (GPIO23); no longer U1.38 (GPIO26_ADC0)
- net M_S3: now also U1.36 (GPIO24); no longer U1.37 (GPIO25)
- net M_S4: now also U1.37 (GPIO25); no longer U1.36 (GPIO24)
- net M_S5: now also U1.38 (GPIO26_ADC0); no longer U1.35 (GPIO23)
- net UART_RX: now reaches U1.16 (GPIO13)
- net UART_RX: now also J11.1 (Pin_1)
- net UART_TX: now reaches U1.27 (GPIO16)
- net UART_TX: now also J11.2 (Pin_2)
- no-connect marks 2 -> 3

Commit message: final tweaks, as sent to fab
Parts:
- J14: digikey SAM1156-01-ND -> 952-3598-ND
- J2: LCSC (none) -> C5885449
- J4: digikey (none) -> 455-1706-ND
Changed lines of the file:
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@@
 			)
 		)
-		(property "digikey" "SAM1156-01-ND"
+		(property "digikey" "952-3598-ND"
 			(at 100.33 49.53 90)
 			(hide yes)
@@
 			)
 		)
+		(property "LCSC" "C5885449"
+			(at 92.71 140.97 0)
+			(hide yes)
+			(show_name no)
+			(do_not_autoplace no)
+			(effects
+				(font
+					(size 1.27 1.27)
+				)
+			)
+		)
 		(pin "10"
 		)
@@
 			(at 256.54 80.01 0)
 			(hide yes)
+			(show_name no)
+			(do_not_autoplace no)
+			(effects
+				(font
+					(size 1.27 1.27)
+				)
+			)
+		)
+		(property "digikey" "455-1706-ND"
+			(at 256.54 80.01 0)
+			(hide yes)
