File: beavs-6.kicad_pcb (KiCad board)
At the start: 4 copper layers, 50 x 70 mm, 134 parts, among them J1 USB_C_Receptacle_USB2.0_16P, J10 Conn_01x03, J11 Conn_01x03, J12 Micro_SD_Card, J13 Conn_02x02_Odd_Even, J14 Conn_01x02, J2 Conn_Coaxial, J3 Conn_01x02, J4 Conn_Coaxial, J5 Conn_01x02, J6 Conn_01x03, J7 Conn_01x03, J8 Conn_01x03, J9 Conn_01x03, Q1 CSD17575Q3, Q2 CSD17575Q3, SW1 SW_Push, SW2 SW_Push, U1 RP2040, U10 INA745A, U11 INA745A, U12 INA745A, U13 INA745A, U14 ISM6HG256X, U15 SN74LVC4245APW, U16 SRV05-4, U17 SRV05-4, U18 LIS2MDL, U19 LM74502, U2 W25Q128JVS, U3 MS5607-02BA, U4 RFM95W-915S2, U5 MAX-M10S, U6 INA745A, U7 AMS1117-3.3, U8 AMS1117-5.0, U9 INA745A, Y1 Crystal_GND24

Commit message: changes!
Parts:
- removed C22: 100n, Capacitor_SMD:C_0402_1005Metric
- removed C45, C46: 220n, Capacitor_SMD:C_0402_1005Metric
- removed D10: LED, LED_SMD:LED_0805_2012Metric
- removed D11: D_Schottky, Diode_SMD:D_SOD-123
- removed D17: D_Zener, Diode_SMD:Nexperia_CFP3_SOD-123W
- removed J11: Conn_01x03, beavs-footprints:JST_VH_B3P-VH-B_1x03_P3.96mm_Vertical_model
- removed J13: Conn_02x02_Odd_Even, Connector_PinHeader_1.27mm:PinHeader_2x02_P1.27mm_Vertical
- removed Q1, Q2: CSD17575Q3, beavs-footprints:SON-8-1EP-3.3x3.3mm-nexfet
- removed R11: 1k, Resistor_SMD:R_0402_1005Metric
- removed R15: 5.1k, Resistor_SMD:R_0402_1005Metric
- removed R2: 300, Resistor_SMD:R_1206_3216Metric
- removed the REF** at (203.0, 63.1)
- removed TP1, TP2: TestPoint, TestPoint:TestPoint_Pad_D1.0mm
- removed U13: INA745A, beavs-footprints:QFN-14-REL_TI
- removed U19: LM74502, beavs-footprints:SOT-23-8-THIN
- removed U5: MAX-M10S, RF_GPS:ublox_MAX
- removed kibuzzard-6945FAFA: G***, kibuzzard-6945FAFA
- added JP1: Jumper_2_Open, Resistor_SMD:R_0402_1005Metric, F.Cu at (219.9, 62.6)
- J2: value Conn_Coaxial -> Conn_ARM_JTAG_SWD_10; footprint Connector_Coaxial:U.FL_Hirose_U.FL-R-SMT-1_Vertical -> Connector_PinHeader_1.27mm:PinHeader_2x05_P1.27mm_Vertical_SMD
- J4: value Conn_Coaxial -> Conn_01x04; footprint Connector_Coaxial:U.FL_Hirose_U.FL-R-SMT-1_Vertical -> Connector_JST:JST_PH_B4B-PH-K_1x04_P2.00mm_Vertical
- U4: value RFM95W-915S2 -> TPS25983; footprint RF_Module:HOPERF_RFM9XW_SMD -> beavs-footprints:Texas_RGE0024M_QFN-24_4x4_Pitch0.5mm_2EP
- moved J4 52.0 mm to (217.8, 108.0), turned to 0 degrees
- moved R8 30.0 mm to (232.0, 79.5), turned to 0 degrees
- moved U15 28.6 mm to (209.7, 67.2), turned to 0 degrees
- moved R9 28.3 mm to (231.0, 82.7), turned to 0 degrees
- moved SW2 28.1 mm to (202.2, 56.9)
- moved U16 25.3 mm to (210.1, 60.8)
- moved R10 24.4 mm to (204.4, 89.0), turned to 180 degrees
- moved Y1 23.8 mm to (225.1, 81.3), turned to -90 degrees
- moved C2 22.6 mm to (225.1, 84.0), turned to 0 degrees
- moved U4 22.1 mm to (193.4, 61.2), turned to -90 degrees
- moved C1 22.1 mm to (225.7, 78.7)
- moved SW1 21.9 mm to (205.8, 56.9), turned to -90 degrees
- moved R1 20.4 mm to (222.9, 80.0)
- moved U17 20.2 mm to (207.5, 74.0)
- moved C9 19.4 mm to (219.7, 74.7), turned to 0 degrees
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Connections:
- J2 pad 1: Net-(J2-In) -> +3V3
- J2 pad 2: GND -> Net-(J2-SWDIO/TMS)
- J4 pad 1: Net-(J4-In) -> +3V3
- J4 pad 2: GND -> unconnected-(J4-Pin_2-Pad2)
- U1 pad 11: /Power/EN -> /SD Card/DAT0
- U1 pad 12: MOSI -> /SD Card/DAT1
- U1 pad 13: MISO -> /SD Card/DAT2
- U1 pad 14: SCK -> /SD Card/DAT3
- U1 pad 15: /mcu/M_LED_D -> /SD Card/CLK
- U1 pad 16: /Sensors/BARO_CS -> unconnected-(U1-GPIO13-Pad16)
- U1 pad 17: /Sensors/IMU_CS -> unconnected-(U1-GPIO14-Pad17)
- U1 pad 18: Net-(J13-Pin_1) -> unconnected-(U1-GPIO15-Pad18)
- U1 pad 2: /Radio/CS -> MISO
- U1 pad 24: Net-(U1-SWCLK) -> Net-(J2-SWCLK/TCK)
- U1 pad 25: Net-(U1-SWD) -> Net-(J2-SWDIO/TMS)
- U1 pad 27: /mcu/M_S6 -> unconnected-(U1-GPIO16-Pad27)
- U1 pad 28: /mcu/M_S5 -> unconnected-(U1-GPIO17-Pad28)
- U1 pad 29: /SD Card/CMD -> unconnected-(U1-GPIO18-Pad29)
- U1 pad 3: /Radio/D0 -> /Sensors/BARO_CS
- U1 pad 30: /SD Card/DAT0 -> unconnected-(U1-GPIO19-Pad30)
- U1 pad 31: /SD Card/DAT1 -> unconnected-(U1-GPIO20-Pad31)
- U1 pad 32: /SD Card/DAT2 -> unconnected-(U1-GPIO21-Pad32)
- U1 pad 34: /SD Card/DAT3 -> /mcu/LEVELSHIFT_DIR
- U1 pad 35: /SD Card/CLK -> /mcu/M_LED_D
- U1 pad 36: /mcu/M_S4 -> /mcu/M_S1
- U1 pad 37: /mcu/M_S3 -> /mcu/M_S2
- U1 pad 38: /mcu/BATTERY_SENSE -> /mcu/M_S3
- U1 pad 39: /Sensors/EXTINT -> /mcu/M_S4
- U1 pad 4: /Radio/RESET -> SCK
- U1 pad 40: /mcu/M_S1 -> /mcu/M_S5
- U1 pad 41: /mcu/M_S2 -> /mcu/BATTERY_SENSE
- U1 pad 5: /mcu/LEVELSHIFT_DIR -> MOSI
- U1 pad 8: /ARM_SWITCH -> /Sensors/IMU_CS
- U1 pad 9: Net-(J13-Pin_3) -> /SD Card/CMD
- U15 pad 15: /mcu/M_S1 -> /mcu/M_S5
- U15 pad 16: /mcu/M_S2 -> /mcu/M_S4
- U15 pad 18: /mcu/M_S4 -> /mcu/M_S2
- U15 pad 19: /mcu/M_S5 -> /mcu/M_S1
- U15 pad 20: /mcu/M_S6 -> GND
- U15 pad 4: /servos/S6 -> unconnected-(U15-A2-Pad4)
- U15 pad 5: /servos/S5 -> /servos/S1
- U15 pad 6: /servos/S4 -> /servos/S2
- U15 pad 8: /servos/S2 -> /servos/S4
- U15 pad 9: /servos/S1 -> /servos/S5
- U16 pad 1: /servos/S1 -> /servos/S5
- U16 pad 3: /servos/S2 -> /servos/S4
- U17 pad 1: /servos/S6 -> unconnected-(U17-IO1-Pad1)
- U17 pad 3: /servos/S4 -> /servos/S2
- U17 pad 6: /servos/S5 -> /servos/S1
- U4 pad 1: GND -> Net-(D7-A)
- U4 pad 10: GND -> unconnected-(U4-RETRY_DLY-Pad10)
- U4 pad 13: +3V3 -> unconnected-(U4-PG-Pad13)
- U4 pad 14: /Radio/D0 -> GND
- U4 pad 16: unconnected-(U4-DIO2-Pad16) -> Net-(D7-A)
- U4 pad 2: MISO -> Net-(D7-A)
- U4 pad 3: MOSI -> Net-(D7-A)
- U4 pad 4: SCK -> GND
- U4 pad 5: /Radio/CS -> GND
- U4 pad 6: /Radio/RESET -> unconnected-(U4-EN/UVLO-Pad6)
- U4 pad 8: GND -> unconnected-(U4-ILIM-Pad8)
- U4 pad 9: Net-(J4-In) -> unconnected-(U4-IMON-Pad9)
Routing:
- net SCL: track 117.2 -> 0.00 mm, vias 10 -> 0
- net SDA: track 116.7 -> 0.00 mm, vias 10 -> 0
- net +5V: track 100.1 -> 0.00 mm, vias 8 -> 0
- net /servos/S6: track 89.6 -> 0.00 mm, vias 4 -> 0
- net SCK: track 83.4 -> 0.00 mm, vias 5 -> 0
- net MOSI: track 82.6 -> 0.00 mm, vias 5 -> 0
- net /servos/S5: track 81.8 -> 0.00 mm, vias 4 -> 0
- net MISO: track 78.0 -> 0.00 mm, vias 5 -> 0
- net /servos/S4: track 70.3 -> 0.00 mm, vias 4 -> 0
- net /servos/S1: track 67.0 -> 0.00 mm, vias 3 -> 0
- net /servos/S2: track 64.1 -> 0.00 mm, vias 3 -> 0
- net /servos/S3: track 59.8 -> 0.00 mm, vias 2 -> 0
- net VBUS: track 57.0 -> 0.00 mm, vias 3 -> 0
- net /mcu/~{RESET}: track 52.3 -> 1.14 mm, vias 2 -> 1
- net /Radio/RESET: track 46.6 -> 0.00 mm, vias 2 -> 0
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- added copper zone on F.Cu, net Net-(D7-K)
- removed copper zone on B.Cu, net Net-(D17-K)
- removed copper zone on F.Cu, net Net-(D17-K)
- removed copper zone on F.Cu, net Net-(U19-SRC)
Other:
- board text removed: "Status"

Commit message: relayout and route
Parts:
- removed D6: SK6812-EC20, beavs-footprints:LED_SK6812-EC20_PLCC4_2.0x2.0mm
- removed NT5, NT6: NetTie_2, NetTie:NetTie-2_SMD_Pad2.0mm
- removed U16, U17: SRV05-4, Package_TO_SOT_SMD:SOT-23-6
- removed kibuzzard-69309731: G***, kibuzzard-69309731
- removed kibuzzard-6945FC37: G***, kibuzzard-6945FC37
- added C22: 100n, Capacitor_SMD:C_0402_1005Metric, F.Cu at (189.7, 82.2)
- added kibuzzard-6ACD650F: G***, kibuzzard-6ACD650F, F.Cu at (180.4, 77.4)
- added kibuzzard-6ACD6545: G***, kibuzzard-6ACD6545, F.Cu at (194.3, 101.3)
- NT2: moved to F.Cu
- NT3, NT4: moved to B.Cu
- moved D7 58.9 mm to (193.3, 61.5), turned to 0 degrees
- moved D8 54.3 mm to (189.5, 62.6), turned to 90 degrees
- moved R8 48.0 mm to (204.6, 118.9), turned to -90 degrees
- moved R7 44.3 mm to (193.3, 59.8), turned to 180 degrees
- moved R9 44.2 mm to (205.6, 118.9), turned to -90 degrees
- moved R6 43.4 mm to (195.2, 59.8), turned to 180 degrees
- moved J1 41.8 mm to (181.2, 65.8), turned to -90 degrees
- moved D1 40.3 mm to (200.0, 101.5)
- moved kibuzzard-6945FB0B 39.9 mm to (215.1, 114.9), turned to 0 degrees
- moved D2 39.5 mm to (200.0, 104.2)
- moved kibuzzard-6945FB1F 39.2 mm to (215.1, 93.1), turned to 0 degrees
- moved C28 39.2 mm to (185.1, 114.8), turned to 90 degrees
- moved C4 38.8 mm to (181.5, 114.5), turned to 180 degrees
- moved kibuzzard-6930C9FF 38.8 mm to (194.7, 104.0)
- moved kibuzzard-693096D7 38.7 mm to (194.7, 107.0)
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Connections:
- D5 pad 2: Net-(D5-DOUT) -> unconnected-(D5-DOUT-Pad2)
- D7 pad 2: Net-(D7-A) -> VDD
- J3 pad 2: Net-(D7-A) -> VDD
- J4 pad 2: unconnected-(J4-Pin_2-Pad2) -> Net-(J4-Pin_2)
- J4 pad 3: unconnected-(J4-Pin_3-Pad3) -> Net-(J4-Pin_3)
- R6 pad 1: +BATT -> VDD
- U1 pad 17: unconnected-(U1-GPIO14-Pad17) -> Net-(J4-Pin_2)
- U1 pad 18: unconnected-(U1-GPIO15-Pad18) -> Net-(J4-Pin_3)
- U1 pad 28: unconnected-(U1-GPIO17-Pad28) -> /Power/EN
- U1 pad 29: unconnected-(U1-GPIO18-Pad29) -> /mcu/LEVELSHIFT_DIR
- U1 pad 34: /mcu/LEVELSHIFT_DIR -> /mcu/M_LED_D
- U1 pad 35: /mcu/M_LED_D -> /mcu/M_S5
- U1 pad 36: /mcu/M_S1 -> /mcu/M_S4
- U1 pad 37: /mcu/M_S2 -> /mcu/M_S3
- U1 pad 38: /mcu/M_S3 -> /mcu/M_S2
- U1 pad 39: /mcu/M_S4 -> /mcu/M_S1
- U1 pad 40: /mcu/M_S5 -> /ARM_SWITCH
- U15 pad 15: /mcu/M_S5 -> /mcu/M_S1
- U15 pad 16: /mcu/M_S4 -> /mcu/M_S2
- U15 pad 18: /mcu/M_S2 -> /mcu/M_S4
- U15 pad 19: /mcu/M_S1 -> /mcu/M_S5
- U15 pad 5: /servos/S1 -> /servos/S5
- U15 pad 6: /servos/S2 -> /servos/S4
- U15 pad 8: /servos/S4 -> /servos/S2
- U15 pad 9: /servos/S5 -> /servos/S1
- U4 pad 1: Net-(D7-A) -> VDD
- U4 pad 12: unconnected-(U4-OVLO-Pad12) -> GND
- U4 pad 16: Net-(D7-A) -> VDD
- U4 pad 2: Net-(D7-A) -> VDD
- U4 pad 25: Net-(D7-A) -> VDD
- U4 pad 3: Net-(D7-A) -> VDD
- U4 pad 6: unconnected-(U4-EN/UVLO-Pad6) -> /Power/EN
Routing:
- net SCL: track 0.00 -> 115.9 mm, vias 0 -> 8
- net SDA: track 0.00 -> 114.8 mm, vias 0 -> 8
- net Net-(D7-A): track 81.1 -> 0.00 mm, vias 2 -> 0
- net +5V: track 0.00 -> 73.6 mm, vias 0 -> 6
- net Net-(D7-K): track 9.19 -> 74.9 mm, vias 2 -> 4
- net /mcu/~{RESET}: track 1.14 -> 53.9 mm, vias 1 -> 4
- net MOSI: track 0.00 -> 51.0 mm, vias 0 -> 4
- net SCK: track 0.00 -> 50.6 mm, vias 0 -> 4
- net MISO: track 0.00 -> 48.3 mm, vias 0 -> 4
- net /Sensors/IMU_CS: track 0.00 -> 48.2 mm, vias 0 -> 4
- net /servos/S5: track 0.00 -> 47.5 mm, vias 0 -> 1
- net Net-(J4-Pin_2): track 0.00 -> 46.1 mm, vias 0 -> 2
- net Net-(J4-Pin_3): track 0.00 -> 44.7 mm, vias 0 -> 2
- net /servos/S4: track 0.00 -> 36.8 mm, vias 0 -> 1
- net +3V3: track 8.67 -> 44.0 mm, vias 0 -> 28
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- added copper zone on B.Cu, net VDD
- added copper zone on F.Cu, net VDD
- removed copper zone on B.Cu, net Net-(D7-A)
- removed copper zone on F.Cu, net Net-(D7-A)
- removed copper zone on F.Cu, net Net-(D7-K)
Other:
- board text added: "BEAVS 6.7"
- board text removed: "BEAVS 6.0"

Commit message: add reverse polarity protection
Parts:
- added C32: 100n, Capacitor_SMD:C_0603_1608Metric, F.Cu at (211.2, 55.1)
- added Q1: Q_NMOS_SSSGD_AvalancheRated, Package_SO:Vishay_PowerPAK_1212-8_Single, F.Cu at (208.7, 58.5)
- added R2: 2k, Resistor_SMD:R_0402_1005Metric, F.Cu at (214.8, 62.5)
- added U5: LM74700, Package_TO_SOT_SMD:SOT-23-6, F.Cu at (208.4, 55.0)
- moved U4 10.1 mm to (218.0, 62.7)
- moved REF** 0.64 mm to (212.9, 55.5)
Connections:
- D7 pad 2: VDD -> Net-(D7-A)
- J3 pad 2: VDD -> Net-(D7-A)
- U1 pad 32: unconnected-(U1-GPIO21-Pad32) -> /ARM_SWITCH
- U1 pad 40: /ARM_SWITCH -> unconnected-(U1-GPIO28_ADC2-Pad40)
- U4 pad 11: unconnected-(U4-NRETRY-Pad11) -> GND
- U4 pad 8: unconnected-(U4-ILIM-Pad8) -> Net-(U4-ILIM)
Routing:
- net VDD: track 12.0 -> 1.84 mm
- net unconnected-(U1-GPIO28_ADC2-Pad40): track 0.00 -> 7.18 mm, vias 0 -> 2
- net Net-(Q1-G): track 0.00 -> 6.77 mm, vias 0 -> 2
- net Net-(D7-A): track 0.00 -> 5.22 mm
- net /ARM_SWITCH: track 13.9 -> 17.4 mm
- net GND: track 11.0 -> 13.3 mm, vias 27 -> 28
- net Net-(U5-VCAP): track 0.00 -> 1.69 mm
- net Net-(U4-ILIM): track 0.00 -> 1.27 mm
- net /Power/EN: track 26.7 -> 27.6 mm
- net unconnected-(U4-IMON-Pad9): track 0.00 -> 0.61 mm, vias 0 -> 1
- added copper zone on F.Cu, net Net-(D7-A)

Commit message: restore symbols library, wire up PG and IMON, refine routing
Parts:
- added C33: 1n, Capacitor_SMD:C_0402_1005Metric, F.Cu at (214.9, 64.3)
- added C34: TBD, Capacitor_SMD:C_0402_1005Metric, F.Cu at (214.5, 61.2)
- added C35: 10u, Capacitor_SMD:C_0603_1608Metric, F.Cu at (217.9, 66.0)
- added R11: 33, Resistor_SMD:R_0402_1005Metric, F.Cu at (212.4, 62.2)
- added R15: 51k, Resistor_SMD:R_0402_1005Metric, F.Cu at (197.4, 72.3)
- added R16: 510, Resistor_SMD:R_0402_1005Metric, F.Cu at (210.5, 62.2)
- R2: value 2k -> 49.9
- moved C21 2.50 mm to (218.1, 94.8)
- moved U10 2.50 mm to (217.5, 92.4)
- moved kibuzzard-6945FB30 2.20 mm to (213.6, 63.8)
- moved C20 2.00 mm to (218.1, 81.8)
- moved U9 2.00 mm to (217.5, 79.3)
- moved C30 1.90 mm to (218.4, 74.5)
- moved C27 1.60 mm to (218.1, 85.5)
- moved C19 1.00 mm to (217.8, 71.2)
- moved U6 1.00 mm to (217.4, 68.7)
- moved R2 0.62 mm to (214.3, 62.2), turned to 0 degrees
- moved C9 0.10 mm to (194.2, 71.8)
Connections:
- C32 pad 1: Net-(D7-A) -> Net-(J3-Pin_2)
- D7 pad 2: Net-(D7-A) -> VDD
- J3 pad 2: Net-(D7-A) -> Net-(J3-Pin_2)
- Q1 pad 1: Net-(D7-A) -> Net-(J3-Pin_2)
- Q1 pad 2: Net-(D7-A) -> Net-(J3-Pin_2)
- Q1 pad 3: Net-(D7-A) -> Net-(J3-Pin_2)
- R2 pad 1: GND -> Net-(R11-Pad2)
- U1 pad 30: unconnected-(U1-GPIO19-Pad30) -> /Power/PG
- U1 pad 40: unconnected-(U1-GPIO28_ADC2-Pad40) -> /Power/IMON
- U4 pad 13: unconnected-(U4-PG-Pad13) -> /Power/PG
- U4 pad 15: unconnected-(U4-DVDT/BGATE-Pad15) -> Net-(U4-DVDT/BGATE)
- U4 pad 7: unconnected-(U4-ITIMER-Pad7) -> Net-(U4-ITIMER)
- U4 pad 9: unconnected-(U4-IMON-Pad9) -> Net-(U4-IMON)
- U5 pad 3: Net-(D7-A) -> Net-(J3-Pin_2)
- U5 pad 6: Net-(D7-A) -> Net-(J3-Pin_2)
Routing:
- net Net-(U4-IMON): track 0.00 -> 30.9 mm, vias 0 -> 4
- net /Power/PG: track 0.00 -> 29.8 mm, vias 0 -> 3
- net VDD: track 1.84 -> 19.6 mm, vias 1 -> 3
- net unconnected-(U1-GPIO28_ADC2-Pad40): track 7.18 -> 0.00 mm, vias 2 -> 0
- net /Power/IMON: track 0.00 -> 7.18 mm, vias 0 -> 2
- net Net-(J3-Pin_2): track 0.00 -> 5.22 mm
- net Net-(D7-A): track 5.22 -> 0.00 mm
- net Net-(U4-DVDT/BGATE): track 0.00 -> 3.95 mm, vias 0 -> 2
- net GND: track 13.3 -> 16.8 mm, vias 28 -> 29
- net Net-(U4-ITIMER): track 0.00 -> 1.33 mm
- net GND1: track 0.00 -> 1.01 mm
- net Net-(R11-Pad2): track 0.00 -> 0.89 mm
- net SDA: track 114.8 -> 114.2 mm
- net unconnected-(U4-IMON-Pad9): track 0.61 -> 0.00 mm, vias 1 -> 0
- added copper zone on F.Cu, net Net-(J3-Pin_2)
- removed copper zone on F.Cu, net Net-(D7-A)
