File: beavs-6.kicad_pcb (KiCad board)
At the start: 4 copper layers, 50 x 70 mm, 121 parts, among them J1 USB_C_Receptacle_USB2.0_16P, J10 Conn_01x03, J12 Micro_SD_Card, J14 Conn_01x02, J2 Conn_ARM_JTAG_SWD_10, J3 Conn_01x02, J4 Conn_01x04, J5 Conn_01x02, J6 Conn_01x03, J7 Conn_01x03, J8 Conn_01x03, J9 Conn_01x03, Q1 Q_NMOS_SSSGD_AvalancheRated, SW1 SW_Push, SW2 SW_Push, U1 RP2040, U10 INA745A, U11 INA745A, U12 INA745A, U14 ISM6HG256X, U15 SN74LVC4245APW, U18 LIS2MDL, U2 W25Q128JVS, U3 MS5607-02BA, U4 TPS25983, U5 LM74700, U6 INA745A, U7 AMS1117-3.3, U8 AMS1117-5.0, U9 INA745A, Y1 Crystal_GND24

Commit message: mostly cosmetic changes
Parts:
- removed kibuzzard-6ACD6545: G***, kibuzzard-6ACD6545
- added J11: Conn_01x03, Connector_PinHeader_2.54mm:PinHeader_1x03_P2.54mm_Vertical, F.Cu at (208.0, 121.1)
- added NT5: NetTie_2, NetTie:NetTie-2_SMD_Pad0.5mm, F.Cu at (208.0, 63.0)
- added NT6: NetTie_2, NetTie:NetTie-2_SMD_Pad0.5mm, F.Cu at (207.6, 63.0)
- added R17: 56k, Resistor_SMD:R_0402_1005Metric, F.Cu at (187.6, 63.9)
- added R18: 56k, Resistor_SMD:R_0402_1005Metric, F.Cu at (187.4, 65.3)
- added REF**: Smolhaj_Scale_0.1, Symbol:Smolhaj_Scale_0.1, B.Cu at (193.4, 55.9)
- added kibuzzard-6ACFDF65: G***, kibuzzard-6ACFDF65, F.Cu at (194.1, 101.5)
- moved kibuzzard-6945FB28 5.28 mm to (213.6, 75.4)
- moved kibuzzard-6945FB1F 4.30 mm to (214.9, 88.8)
- moved D12 2.16 mm to (209.7, 69.6), turned to 180 degrees
- moved R8 1.40 mm to (203.3, 118.4), turned to 0 degrees
- moved REF** 1.33 mm to (222.3, 97.3)
- moved R9 0.64 mm to (205.2, 118.4), turned to 180 degrees
- moved NT2 0.59 mm to (206.2, 62.8)
- moved kibuzzard-69309760 0.52 mm to (195.1, 112.5)
- moved kibuzzard-6945FB0B 0.50 mm to (214.8, 115.3)
- moved R3 0.35 mm to (186.6, 63.9)
- moved D13 0.32 mm to (210.0, 81.5)
- moved kibuzzard-6930C9FF 0.31 mm to (194.6, 104.3)
- moved kibuzzard-6930C9BE 0.31 mm to (195.6, 109.8)
- moved NT4 0.21 mm to (206.0, 62.4)
- moved kibuzzard-693096D7 0.16 mm to (194.9, 107.0)
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Connections:
- U1 pad 16: unconnected-(U1-GPIO13-Pad16) -> /mcu/UART_RX
- U1 pad 27: unconnected-(U1-GPIO16-Pad27) -> /mcu/UART_TX
- U1 pad 35: /mcu/M_S5 -> /mcu/M_S2
- U1 pad 36: /mcu/M_S4 -> /mcu/M_S3
- U1 pad 37: /mcu/M_S3 -> /mcu/M_S4
- U1 pad 38: /mcu/M_S2 -> /mcu/M_S5
- U15 pad 16: /mcu/M_S2 -> /mcu/M_S5
- U15 pad 17: /mcu/M_S3 -> /mcu/M_S4
- U15 pad 18: /mcu/M_S4 -> /mcu/M_S3
- U15 pad 19: /mcu/M_S5 -> /mcu/M_S2
- U15 pad 5: /servos/S5 -> /servos/S2
- U15 pad 6: /servos/S4 -> /servos/S3
- U15 pad 7: /servos/S3 -> /servos/S4
- U15 pad 8: /servos/S2 -> /servos/S5
Routing:
- net /mcu/UART_TX: track 0.00 -> 60.0 mm, vias 0 -> 2
- net /mcu/UART_RX: track 0.00 -> 58.0 mm, vias 0 -> 2
- net +5V: track 73.6 -> 85.6 mm, vias 6 -> 5
- net Net-(R10-Pad2): track 26.0 -> 31.9 mm
- net /servos/S5: track 47.5 -> 51.6 mm
- net Net-(J1-CC2): track 1.69 -> 4.64 mm, vias 0 -> 2
- net /servos/S4: track 36.8 -> 39.2 mm
- net /mcu/M_S5: track 7.35 -> 9.62 mm
- net /mcu/M_S2: track 9.62 -> 7.35 mm
- net /servos/S2: track 15.4 -> 13.2 mm
- net Net-(D7-K): track 74.9 -> 76.8 mm
- net /Sensors/BARO_CS: track 29.5 -> 31.2 mm
- net /mcu/BATTERY_SENSE: track 21.8 -> 20.6 mm
- net Net-(D1-DIN): track 34.2 -> 35.4 mm
- net Net-(J1-CC1): track 1.90 -> 2.73 mm
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Other:
- board text added: "GND TX RX"
- board text added: "Our Smuckie, who art in Rogers, hallowed be thy name. Thy exam grades come, thy regrades be done, on canvas as they are in gradescope. Give us this our daily lecture, and forgive our mistakes as we forgive your smuckie moments. Lead us not into ignorance but deliver our GPAs from evil. For yours is the power and the glory forever. ABen"
- board text removed: "Our Smuckie, who art in Rogers, hallowed by thy name. Thy exam grades come, thy regrades be done, on canvas as they are in gradescope. Give us this our daily lecture, and forgive our mistakes as we forgive your smuckie moments. Lead us not into ignorance but deliver our GPAs from evil. For yours is the power and the glory forever. ABen"
- board text removed: "SCRT"
