File: beavs-6.kicad_pcb (KiCad board)
At the start: 4 copper layers, 50 x 70 mm, 127 parts, among them J1 USB_C_Receptacle_USB2.0_16P, J10 Conn_01x03, J11 Conn_01x03, J12 Micro_SD_Card, J14 Conn_01x02, J2 Conn_ARM_JTAG_SWD_10, J3 Conn_01x02, J4 Conn_01x04, J5 Conn_01x02, J6 Conn_01x03, J7 Conn_01x03, J8 Conn_01x03, J9 Conn_01x03, Q1 Q_NMOS_SSSGD_AvalancheRated, SW1 SW_Push, SW2 SW_Push, U1 RP2040, U10 INA745A, U11 INA745A, U12 INA745A, U14 ISM6HG256X, U15 SN74LVC4245APW, U18 LIS2MDL, U2 W25Q128JVS, U3 MS5607-02BA, U4 TPS25983, U5 LM74700, U6 INA745A, U7 AMS1117-3.3, U8 AMS1117-5.0, U9 INA745A, Y1 Crystal_GND24

Commit message: final tweaks, as sent to fab
Parts:
- added D10: D_Zener, Diode_SMD:D_SOD-523, F.Cu at (200.2, 114.6)
- added D11: D_Zener, Diode_SMD:D_SOD-523, F.Cu at (204.8, 96.1)
- added D17: D_Zener, Diode_SMD:D_SOD-523, F.Cu at (204.7, 84.6)
- added D18: D_Zener, Diode_SMD:D_SOD-523, F.Cu at (203.6, 73.4)
- added D6: D_Zener, Diode_SMD:D_SOD-523, F.Cu at (200.6, 64.7)
- D12, D13, D14, D15, D16: footprint Diode_SMD:Nexperia_CFP3_SOD-123W -> Diode_SMD:D_SOD-523; moved to F.Cu
- Q1: value Q_NMOS_SSSGD_AvalancheRated -> SIS402DN-T1-GE3
- moved D12 3.42 mm to (209.5, 73.0)
- moved D16 2.96 mm to (210.4, 118.5)
- moved D15 2.93 mm to (210.3, 107.1)
- moved D13 2.91 mm to (210.2, 84.4)
- moved D14 2.81 mm to (210.3, 95.7)
- moved REF** 0.51 mm to (212.5, 121.1)
- moved J5 0.15 mm to (179.6, 73.4)
Routing:
- net /servos/S3: track 26.7 -> 32.0 mm
- net /servos/S2: track 13.2 -> 18.3 mm
- net /servos/S4: track 39.2 -> 44.3 mm
- net Net-(D16-K): track 0.00 -> 4.04 mm
- net /servos/S5: track 51.6 -> 55.5 mm
- net GND1: track 1.01 -> 4.29 mm
- net Net-(D12-K): track 0.00 -> 2.20 mm
- net Net-(D13-K): track 0.00 -> 1.94 mm
- net Net-(D15-K): track 0.00 -> 1.10 mm
- net /servos/S1: track 5.88 -> 6.71 mm
- net /mcu/UART_RX: vias 2 -> 1
- net GND: vias 286 -> 288
- net /mcu/UART_TX: vias 2 -> 1
