File: servos.kicad_sch (KiCad schematic)
At the start: 33 parts, among them J10 Conn_01x03, J11 Conn_01x03, J6 Conn_01x03, J7 Conn_01x03, J8 Conn_01x03, J9 Conn_01x03, U10 INA745A, U11 INA745A, U12 INA745A, U13 INA745A, U6 INA745A, U9 INA745A

Commit message: remove unneeded stuff
Parts:
- removed C22: 100n, Capacitor_SMD:C_0402_1005Metric, symbol Device:C_Small
- removed D17: D_Zener, Diode_SMD:Nexperia_CFP3_SOD-123W, symbol Device:D_Zener
- removed J11: Conn_01x03, beavs-footprints:JST_VH_B3P-VH-B_1x03_P3.96mm_Vertical_model, symbol Connector_Generic:Conn_01x03
- removed U13: INA745A, beavs-footprints:QFN-14-REL_TI, symbol beavs-symbols:INA745

Commit message: relayout and route
Parts:
- removed NT5, NT6: NetTie_2, NetTie:NetTie-2_SMD_Pad2.0mm, symbol Device:NetTie_2

Commit message: mostly cosmetic changes
Parts:
- added NT5, NT6: NetTie_2, NetTie:NetTie-2_SMD_Pad0.5mm, symbol Device:NetTie_2
Connections:
- net GND: now also NT5.2, NT6.2
- net GND1: now also NT5.1, NT6.1
