File: servos.kicad_sch (KiCad schematic)
At the start: 29 parts, among them J10 Conn_01x03, J6 Conn_01x03, J7 Conn_01x03, J8 Conn_01x03, J9 Conn_01x03, U10 INA745A, U11 INA745A, U12 INA745A, U6 INA745A, U9 INA745A

Commit message: final tweaks, as sent to fab
Parts:
- D12, D13, D14, D15, D16: footprint Diode_SMD:Nexperia_CFP3_SOD-123W -> Diode_SMD:D_SOD-523; LCSC (none) -> C20615819; digikey 1727-5361-1-ND -> (none)
Changed lines of the file:
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@@
 			)
 		)
-		(property "Footprint" "Diode_SMD:Nexperia_CFP3_SOD-123W"
+		(property "Footprint" "Diode_SMD:D_SOD-523"
 			(at 167.64 125.73 0)
 			(hide yes)
@@
 			)
 		)
-		(property "digikey" "1727-5361-1-ND"
+		(property "digikey" ""
 			(at 167.64 125.73 90)
 			(hide yes)
@@
 			)
 		)
+		(property "LCSC" "C20615819"
+			(at 167.64 125.73 90)
+			(hide yes)
+			(show_name no)
+			(do_not_autoplace no)
+			(effects
+				(font
+					(size 1.27 1.27)
+				)
+			)
+		)
 		(pin "2"
 		)
@@
 			)
 		)
-		(property "Footprint" "Diode_SMD:Nexperia_CFP3_SOD-123W"
+		(property "Footprint" "Diode_SMD:D_SOD-523"
 			(at 87.63 124.46 0)
 			(hide yes)
@@
 			)
 		)
-		(property "digikey" "1727-5361-1-ND"
+		(property "digikey" ""
 			(at 87.63 124.46 90)
 			(hide yes)
@@
 			)
 		)
+		(property "LCSC" "C20615819"
+			(at 87.63 124.46 90)
+			(hide yes)
+			(show_name no)
+			(do_not_autoplace no)
+			(effects
+				(font
+					(size 1.27 1.27)
+				)
+			)
+		)
 		(pin "2"
 		)
@@
 			)
 		)
-		(property "Footprint" "Diode_SMD:Nexperia_CFP3_SOD-123W"
+		(property "Footprint" "Diode_SMD:D_SOD-523"
 			(at 87.63 64.77 0)
 			(hide yes)
@@
 			)
 		)
-		(property "digikey" "1727-5361-1-ND"
+		(property "digikey" ""
 			(at 87.63 64.77 90)
 			(hide yes)
@@
 			)
 		)
+		(property "LCSC" "C20615819"
+			(at 87.63 64.77 90)
+			(hide yes)
+			(show_name no)
+			(do_not_autoplace no)
+			(effects
+				(font
+					(size 1.27 1.27)
+				)
+			)
+		)
 		(pin "2"
 		)
@@
 			)
 		)
-		(property "Footprint" "Diode_SMD:Nexperia_CFP3_SOD-123W"
+		(property "Footprint" "Diode_SMD:D_SOD-523"
 			(at 246.38 64.77 0)
 			(hide yes)
@@
 			)
 		)
-		(property "digikey" "1727-5361-1-ND"
+		(property "digikey" ""
 			(at 246.38 64.77 90)
 			(hide yes)
@@
 			)
 		)
+		(property "LCSC" "C20615819"
+			(at 246.38 64.77 90)
+			(hide yes)
+			(show_name no)
+			(do_not_autoplace no)
+			(effects
+				(font
+					(size 1.27 1.27)
+				)
+			)
+		)
 		(pin "2"
 		)
@@
 			)
 		)
-		(property "Footprint" "Diode_SMD:Nexperia_CFP3_SOD-123W"
+		(property "Footprint" "Diode_SMD:D_SOD-523"
 			(at 166.37 64.77 0)
 			(hide yes)
@@
 			)
 		)
-		(property "digikey" "1727-5361-1-ND"
+		(property "digikey" ""
 			(at 166.37 64.77 90)
 			(hide yes)
@@
 			(at 166.37 64.77 90)
 			(hide yes)
+			(show_name no)
+			(do_not_autoplace no)
+			(effects
+				(font
+					(size 1.27 1.27)
+				)
+			)
+		)
+		(property "LCSC" "C20615819"
+			(at 166.37 64.77 90)
+			(hide yes)
