File: power.kicad_sch (KiCad schematic)
At the start: 20 parts, among them J3 Conn_01x02, Q1 Q_NMOS_SSSGD_AvalancheRated, U4 TPS25983, U5 LM74700, U7 AMS1117-3.3, U8 AMS1117-5.0

Commit message: mostly cosmetic changes
Parts:
- U7, U8: now not fitted
Changed lines of the file:
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@@
 		(on_board yes)
 		(in_pos_files yes)
-		(dnp no)
+		(dnp yes)
 		(fields_autoplaced yes)
 		(property "Reference" "U8"
@@
 		(on_board yes)
 		(in_pos_files yes)
-		(dnp no)
+		(dnp yes)
 		(fields_autoplaced yes)
 		(property "Reference" "U7"

Commit message: final tweaks, as sent to fab
Parts:
- C33: LCSC (none) -> C1523
- Q1: value Q_NMOS_SSSGD_AvalancheRated -> SIS402DN-T1-GE3; LCSC (none) -> C15791
- R11: LCSC (none) -> C25105
- R2: LCSC (none) -> C25120
- U4: LCSC (none) -> C20607218
- U5: LCSC (none) -> C2653623
Changed lines of the file:
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@@
 			)
 		)
+		(property "LCSC" "C1523"
+			(at 222.25 82.55 0)
+			(hide yes)
+			(show_name no)
+			(do_not_autoplace no)
+			(effects
+				(font
+					(size 1.27 1.27)
+				)
+			)
+		)
 		(pin "1"
 		)
@@
 			)
 		)
+		(property "LCSC" "C20607218"
+			(at 205.74 73.66 0)
+			(hide yes)
+			(show_name no)
+			(do_not_autoplace no)
+			(effects
+				(font
+					(size 1.27 1.27)
+				)
+			)
+		)
 		(pin "6"
 		)
@@
 			)
 		)
+		(property "LCSC" "C25120"
+			(at 185.42 81.28 90)
+			(hide yes)
+			(show_name no)
+			(do_not_autoplace no)
+			(effects
+				(font
+					(size 1.27 1.27)
+				)
+			)
+		)
 		(pin "1"
 		)
@@
 			)
 		)
-		(property "Value" "Q_NMOS_SSSGD_AvalancheRated"
+		(property "Value" "SIS402DN-T1-GE3"
 			(at 72.39 59.69 90)
 			(show_name no)
@@
 			)
 		)
+		(property "LCSC" "C15791"
+			(at 72.39 66.04 90)
+			(hide yes)
+			(show_name no)
+			(do_not_autoplace no)
+			(effects
+				(font
+					(size 1.27 1.27)
+				)
+			)
+		)
 		(pin "4"
 		)
@@
 			)
 		)
+		(property "LCSC" "C25105"
+			(at 176.53 81.28 90)
+			(hide yes)
+			(show_name no)
+			(do_not_autoplace no)
+			(effects
+				(font
+					(size 1.27 1.27)
+				)
+			)
+		)
 		(pin "1"
 		)
@@
 			(at 72.39 81.28 0)
 			(hide yes)
+			(show_name no)
+			(do_not_autoplace no)
+			(effects
+				(font
+					(size 1.27 1.27)
+				)
+			)
+		)
+		(property "LCSC" "C2653623"
+			(at 72.39 81.28 0)
+			(hide yes)
